File: JAWS65.kicad_pcb (KiCad board)
At the start: 2 copper layers, 303.8 x 94.2 mm, 161 parts, among them J1 JST SH 4-pin, J2 AVR-ISP-6, SW1 Reset, U1 SRV05-4, U2 ATmega32U4-AU, Y1 16MHz

Commit message: Added Hotswap + 2 MCU layouts
Parts:
- removed the D14 at (247.1, 9.79)
- removed the D67 at (267.8, 86.0)
- removed the MX14 at (256.6, 9.00)
- removed the MX15 at (275.7, 9.00)
- removed the MX33 at (11.4, 47.1)
- removed the MX62 at (13.8, 85.2)
- removed the MX63 at (37.6, 85.2)
- removed the MX64 at (61.4, 85.2)
- removed the MX65 at (142.3, 85.2)
- removed the MX67 at (223.3, 85.2)
- removed MX69: 1u, MX_Only:MXOnly-1U-NoLED
- added D65: 1N4148, Diode_SMD:D_SOD-123, B.Cu at (256.9, 98.6)
- added MX66: 1u, MX_Only:MXOnly-1U-Hotswap, F.Cu at (283.3, 95.7)
- J2: footprint bakeneko:ISP -> local:ISP; moved to F.Cu
- MX1, MX10, MX11, MX12, MX13, MX2, MX3, MX4, MX5, MX6, MX7, MX8, MX9: footprint MX_Only:MXOnly-1U-NoLED -> MX_Only:MXOnly-1U-Hotswap
- MX14: renamed from MX17; footprint MX_Only:MXOnly-2U-NoLED -> MX_Only:MXOnly-2U-Hotswap
- MX15: renamed from MX16; footprint MX_Only:MXOnly-1U-NoLED -> MX_Only:MXOnly-1U-Hotswap
- MX16: renamed from MX18; footprint MX_Only:MXOnly-1.5U-NoLED -> MX_Only:MXOnly-1.5U-Hotswap
- MX17: renamed from MX19; footprint MX_Only:MXOnly-1U-NoLED -> MX_Only:MXOnly-1U-Hotswap
- MX18: renamed from MX20; footprint MX_Only:MXOnly-1U-NoLED -> MX_Only:MXOnly-1U-Hotswap
- MX19: renamed from MX21; footprint MX_Only:MXOnly-1U-NoLED -> MX_Only:MXOnly-1U-Hotswap
- MX20: renamed from MX22; footprint MX_Only:MXOnly-1U-NoLED -> MX_Only:MXOnly-1U-Hotswap
- MX21: renamed from MX23; footprint MX_Only:MXOnly-1U-NoLED -> MX_Only:MXOnly-1U-Hotswap
- MX22: renamed from MX24; footprint MX_Only:MXOnly-1U-NoLED -> MX_Only:MXOnly-1U-Hotswap
- MX23: renamed from MX25; footprint MX_Only:MXOnly-1U-NoLED -> MX_Only:MXOnly-1U-Hotswap
- MX24: renamed from MX26; footprint MX_Only:MXOnly-1U-NoLED -> MX_Only:MXOnly-1U-Hotswap
- MX25: renamed from MX27; footprint MX_Only:MXOnly-1U-NoLED -> MX_Only:MXOnly-1U-Hotswap
- MX26: renamed from MX28; footprint MX_Only:MXOnly-1U-NoLED -> MX_Only:MXOnly-1U-Hotswap
- MX27: renamed from MX29; footprint MX_Only:MXOnly-1U-NoLED -> MX_Only:MXOnly-1U-Hotswap
- MX28: renamed from MX30; footprint MX_Only:MXOnly-1U-NoLED -> MX_Only:MXOnly-1U-Hotswap
- MX29: renamed from MX31; footprint MX_Only:MXOnly-1.5U-NoLED -> MX_Only:MXOnly-1.5U-Hotswap
- MX30: renamed from MX32; footprint MX_Only:MXOnly-1U-NoLED -> MX_Only:MXOnly-1U-Hotswap
- MX31: renamed from MX34; footprint MX_Only:MXOnly-1.75U-NoLED -> MX_Only:MXOnly-1.75U-Hotswap
- MX32: renamed from MX35; footprint MX_Only:MXOnly-1U-NoLED -> MX_Only:MXOnly-1U-Hotswap
- MX33: renamed from MX36; footprint MX_Only:MXOnly-1U-NoLED -> MX_Only:MXOnly-1U-Hotswap
- MX34: renamed from MX37; footprint MX_Only:MXOnly-1U-NoLED -> MX_Only:MXOnly-1U-Hotswap
- MX35: renamed from MX38; footprint MX_Only:MXOnly-1U-NoLED -> MX_Only:MXOnly-1U-Hotswap
- MX36: renamed from MX39; footprint MX_Only:MXOnly-1U-NoLED -> MX_Only:MXOnly-1U-Hotswap
- MX37: renamed from MX40; footprint MX_Only:MXOnly-1U-NoLED -> MX_Only:MXOnly-1U-Hotswap
- MX38: renamed from MX41; footprint MX_Only:MXOnly-1U-NoLED -> MX_Only:MXOnly-1U-Hotswap
- MX39: renamed from MX42; footprint MX_Only:MXOnly-1U-NoLED -> MX_Only:MXOnly-1U-Hotswap
- MX40: renamed from MX43; footprint MX_Only:MXOnly-1U-NoLED -> MX_Only:MXOnly-1U-Hotswap
- MX41: renamed from MX44; footprint MX_Only:MXOnly-1U-NoLED -> MX_Only:MXOnly-1U-Hotswap
- MX42: renamed from MX45; footprint MX_Only:MXOnly-1U-NoLED -> MX_Only:MXOnly-1U-Hotswap
- MX43: renamed from MX46; footprint MX_Only:MXOnly-2.25U-NoLED -> MX_Only:MXOnly-2.25U-Hotswap
- MX44: renamed from MX47; footprint MX_Only:MXOnly-1U-NoLED -> MX_Only:MXOnly-1U-Hotswap
- MX45: renamed from MX48; footprint MX_Only:MXOnly-2.25U-NoLED -> MX_Only:MXOnly-2.25U-Hotswap
- MX46: renamed from MX49; footprint MX_Only:MXOnly-1U-NoLED -> MX_Only:MXOnly-1U-Hotswap
- MX47: renamed from MX50; footprint MX_Only:MXOnly-1U-NoLED -> MX_Only:MXOnly-1U-Hotswap
- MX48: renamed from MX51; footprint MX_Only:MXOnly-1U-NoLED -> MX_Only:MXOnly-1U-Hotswap
- MX49: renamed from MX52; footprint MX_Only:MXOnly-1U-NoLED -> MX_Only:MXOnly-1U-Hotswap
- MX50: renamed from MX53; footprint MX_Only:MXOnly-1U-NoLED -> MX_Only:MXOnly-1U-Hotswap
- MX51: renamed from MX54; footprint MX_Only:MXOnly-1U-NoLED -> MX_Only:MXOnly-1U-Hotswap
- MX52: renamed from MX55; footprint MX_Only:MXOnly-1U-NoLED -> MX_Only:MXOnly-1U-Hotswap
- MX53: renamed from MX56; footprint MX_Only:MXOnly-1U-NoLED -> MX_Only:MXOnly-1U-Hotswap
- MX54: renamed from MX57; footprint MX_Only:MXOnly-1U-NoLED -> MX_Only:MXOnly-1U-Hotswap
- MX55: renamed from MX58; footprint MX_Only:MXOnly-1U-NoLED -> MX_Only:MXOnly-1U-Hotswap
- MX56: renamed from MX59; footprint MX_Only:MXOnly-1.75U-NoLED -> MX_Only:MXOnly-1.75U-Hotswap
- MX57: renamed from MX60; footprint MX_Only:MXOnly-1U-NoLED -> MX_Only:MXOnly-1U-Hotswap
- MX58: renamed from MX61; footprint MX_Only:MXOnly-1U-NoLED -> MX_Only:MXOnly-1U-Hotswap
- MX59: renamed from MX71; footprint MX_Only:MXOnly-1.25U-NoLED -> MX_Only:MXOnly-1.25U-Hotswap
- MX60: renamed from MX72; footprint MX_Only:MXOnly-1.25U-NoLED -> MX_Only:MXOnly-1.25U-Hotswap
- MX61: renamed from MX73; footprint MX_Only:MXOnly-1.25U-NoLED -> MX_Only:MXOnly-1.25U-Hotswap
- MX62: renamed from MX74; footprint MX_Only:MXOnly-6.25U-ReversedStabilizers-NoLED -> MX_Only:MXOnly-6.25U-Hotswap-ReversedStabilizers
- MX63: renamed from MX66; footprint MX_Only:MXOnly-1.25U-NoLED -> MX_Only:MXOnly-1.25U-Hotswap
- MX64: renamed from MX75; footprint MX_Only:MXOnly-1.25U-NoLED -> MX_Only:MXOnly-1.25U-Hotswap
- MX65: renamed from MX68; footprint MX_Only:MXOnly-1U-NoLED -> MX_Only:MXOnly-1U-Hotswap
- MX67: renamed from MX70; footprint MX_Only:MXOnly-1U-NoLED -> MX_Only:MXOnly-1U-Hotswap
- U2: value ATmega32U4-AU -> ATmega32U4-MUR; footprint Package_QFP:TQFP-44_10x10mm_P0.8mm -> Package_DFN_QFN:QFN-44-1EP_7x7mm_P0.5mm_EP5.2x5.2mm
- moved J2 180.9 mm to (175.0, 83.4), turned to -90 degrees
- moved SW1 146.4 mm to (189.4, 94.1)
- moved C3 145.5 mm to (167.6, 100.0), turned to 180 degrees
- moved C1 145.5 mm to (170.3, 92.6)
- moved C2 145.5 mm to (150.3, 97.2)
- moved C5 145.5 mm to (174.1, 93.5)
- moved C6 145.5 mm to (174.1, 99.1)
- moved R1 145.5 mm to (182.8, 93.2)
- moved Y1 145.5 mm to (174.1, 96.3)
- moved C7 145.4 mm to (161.2, 86.1)
- moved U2 145.4 mm to (161.6, 96.3)
- moved C4 142.7 mm to (153.4, 86.8), turned to -90 degrees
- moved R4 128.2 mm to (150.3, 99.6), turned to 0 degrees
- moved D17 32.5 mm to (37.8, 41.5)
- moved D14 21.3 mm to (266.4, 22.4)
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- renumbered D15 to D14, D16 to D15, D17 to D16, D18 to D17, D19 to D18, D20 to D19, D21 to D20, D22 to D21, D23 to D22, D24 to D23, D25 to D24, D26 to D25, D27 to D26, D28 to D27, D29 to D28, D30 to D29, D31 to D30, D32 to D31, D33 to D32, D34 to D33, D35 to D34, D36 to D35, D37 to D36, D38 to D37, D39 to D38, D40 to D39, D41 to D40, D42 to D41, D43 to D42, D44 to D43, D45 to D44, D46 to D45, D47 to D46, D48 to D47, D49 to D48, D50 to D49, D51 to D50, D52 to D51, D53 to D52, D54 to D53, D55 to D54, D56 to D55, D57 to D56, D58 to D57, D59 to D58, D60 to D59, D61 to D60, D62 to D61, D63 to D62, D64 to D63, D65 to D64, D68 to D67
Connections:
- D66 pad 2: Net-(D66-Pad2) -> Net-(D66-A)
- MX14 pad 2: COL14 -> COL13
- MX15 pad 2: COL15 -> COL14
- MX30 pad 2: COL15 -> COL14
- MX44 pad 2: COL15 -> COL14
- MX58 pad 2: COL15 -> COL14
- MX65 pad 1: Net-(D66-Pad2) -> Net-(D65-A)
- MX67 pad 2: COL15 -> COL14
- U1 pad 3: Net-(U1-Pad3) -> unconnected-(U1-IO2-Pad3)
- U1 pad 4: Net-(U1-Pad4) -> unconnected-(U1-IO3-Pad4)
- U2 pad 1: ROW0 -> COL6
- U2 pad 12: ROW1 -> COL8
- U2 pad 18: COL15 -> ROW0
- U2 pad 19: COL14 -> ROW1
- U2 pad 20: COL13 -> ROW2
- U2 pad 21: COL12 -> ROW3
- U2 pad 22: COL11 -> unconnected-(U2-PD5-Pad22)
- U2 pad 25: COL10 -> COL9
- U2 pad 26: COL9 -> COL10
- U2 pad 27: COL8 -> COL11
- U2 pad 28: COL7 -> COL14
- U2 pad 29: COL6 -> COL13
- U2 pad 30: COL5 -> COL12
- U2 pad 31: COL4 -> unconnected-(U2-PC6-Pad31)
- U2 pad 32: COL3 -> ROW4
- U2 pad 36: ROW2 -> COL0
- U2 pad 37: COL0 -> COL1
- U2 pad 38: ROW4 -> COL2
- U2 pad 39: ROW3 -> COL3
- U2 pad 40: COL2 -> COL4
- U2 pad 41: Net-(U2-Pad41) -> COL5
- U2 pad 42: Net-(U2-Pad42) -> unconnected-(U2-AREF-Pad42)
- U2 pad 8: COL1 -> COL7
Routing:
- net COL15: track 355.0 -> 0.00 mm
- net +5V: track 123.2 -> 307.7 mm, vias 6 -> 9
- net /MCU_D+: track 18.4 -> 189.1 mm
- net /MCU_D-: track 19.2 -> 189.4 mm
- net GND: track 184.5 -> 332.9 mm, vias 5 -> 3
- net COL0: track 99.8 -> 233.6 mm, vias 1 -> 2
- net COL11: track 293.6 -> 175.9 mm, vias 0 -> 8
- net COL9: track 266.7 -> 151.6 mm, vias 0 -> 8
- net COL8: track 217.4 -> 104.0 mm, vias 0 -> 8
- net COL13: track 353.1 -> 241.1 mm, vias 0 -> 8
- net COL7: track 198.8 -> 93.0 mm, vias 0 -> 8
- net COL6: track 212.1 -> 108.1 mm, vias 0 -> 10
- net COL12: track 318.3 -> 214.9 mm, vias 0 -> 8
- net COL10: track 254.7 -> 154.5 mm, vias 0 -> 8
- net COL1: track 113.8 -> 207.2 mm, vias 0 -> 8
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Other:
- board text added: "JAWS65"
- board text removed: "Bakeneko65 v3.0"
